File: Kelly controller.sch (KiCad schematic (older format))
At the start: 16 parts, among them J1 Conn_01x06_Female, J2 Conn_01x06_Female, J4 Meter, J5 48V, J6 12V, J7 5V, SW1 FNR, SW2 Foot Switch, SW3 Brake, SW4 Power Switch

Commit message: first commit on branch base. Incorporates minor change in schematic notes. Base branch will be useful for any fresh starts in the future.
Other:
- note added: "Rev 2: \nTo be used with Kelly assemblies on first prototype vehicle for basic manual control. \nFuture versions will use mcu.\nThis version will be saved as a 'base' branch in git for future reference and development\n\nChanges:\n- Dropped display output \n- Adapted wiring to flat 14 pin connector from assembly\n- Dropped battery connector (superfluous - power comes in on brown line and goes bac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"
- note removed: "Rev 2: \nTo be used with Kelly assemblies on first prototype vehicle for basic manual control. \nFuture versions will use mcu\n\nChanges:\n- Dropped display output \n- Adapted wiring to flat 14 pin connector from assembly\n- Dropped battery connector (superfluous - power comes in on brown line and goes back to \n controller on pink line via power switch)\n- Made 12V line thicker (consistent with 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"
Changed lines of the file:
@@
 make sure boost is not\nenabled in app
 Text Notes 650  7750 0    100  ~ 0
-Rev 2: \nTo be used with Kelly assemblies on first prototype vehicle for basic manual control. \nFuture versions will use mcu\n\nChanges:\n- Dropped display output \n- Adapted wiring to flat 14 pin connector from assembly\n- Dropped battery connector (superfluous - power comes in on brown line and goes back to \n  controller on pink line via power switch)\n- Made 12V line thicker (consistent with thicker wire coming from connector)\n\nTo do:\n- Flip control connectors to face same direction?\n\nURLs:\n- KLS controller manual: https://kellycontroller.com/wp-content/uploads/kls-nm/KellyKLS-N-UserManualV2.7.pdf\n- Control box and assembly schematic: https://kellycontroller.com/wp-content/uploads/kls-h/KLS-DHMN-CAD-Model-1130.pdf\n- Display datasheet: https://drive.google.com/file/d/12TWD7V3HLI8IPtFdbf37xQo0YPuW2e0G/view
+Rev 2: \nTo be used with Kelly assemblies on first prototype vehicle for basic manual control. \nFuture versions will use mcu.\nThis version will be saved as a 'base' branch in git for future reference and development\n\nChanges:\n- Dropped display output \n- Adapted wiring to flat 14 pin connector from assembly\n- Dropped battery connector (superfluous - power comes in on brown line and goes back to \n  controller on pink line via power switch)\n- Made 12V line thicker (consistent with thicker wire coming from connector)\n\nTo do:\n- Flip control connectors to face same direction?\n\nURLs:\n- KLS controller manual: https://kellycontroller.com/wp-content/uploads/kls-nm/KellyKLS-N-UserManualV2.7.pdf\n- Control box and assembly schematic: https://kellycontroller.com/wp-content/uploads/kls-h/KLS-DHMN-CAD-Model-1130.pdf\n- Display datasheet: https://drive.google.com/file/d/12TWD7V3HLI8IPtFdbf37xQo0YPuW2e0G/view
 Text Notes 7750 1750 0    50   ~ 0
 From: https://kellycontroller.com/wp-content/uploads/kls-h/KLS-DHMN-CAD-Model-1130.pdf
