File: Kelly controller.sch (KiCad schematic (older format))
At the start: 19 parts, among them J1 CAN, J2 Kelly1, J3 Display, J4 Kelly2, J5 48V, J6 12V, J7 5V, K1 Contactor, SW1 FNR, SW2 Foot Switch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

Commit message: removed auto connectors and added assembly connector
Parts:
- removed BT1: Battery, TerminalBlock:TerminalBlock_bornier-2_P5.08mm, symbol Device:Battery
- removed J1: CAN, Connector_Molex:Molex_SL_171971-0002_1x02_P2.54mm_Vertical, symbol Connector:Conn_01x02_Female
- removed J2: Kelly1, Connector_Molex:Molex_KK-254_AE-6410-08A_1x08_P2.54mm_Vertical, symbol Connector:Conn_01x08_Female
- removed J3: Display, Connector_Molex:Molex_KK-254_AE-6410-05A_1x05_P2.54mm_Vertical, symbol Connector:Conn_01x05_Female
- removed J4: Kelly2, Connector_Molex:Molex_SL_171971-0007_1x07_P2.54mm_Vertical, symbol Connector:Conn_01x07_Female
- removed K1: Contactor, TerminalBlock:TerminalBlock_bornier-2_P5.08mm, symbol my_devices:RM50-xx21
- added J2: Conn_01x12_Female, Connector_Molex:Molex_SL_171971-0012_1x12_P2.54mm_Vertical, symbol Connector:Conn_01x12_Female
- added J3: Batt, TerminalBlock:TerminalBlock_bornier-2_P5.08mm, symbol Connector:Conn_01x02_Female
- added J4: Meter, Connector_Molex:Molex_SL_171971-0002_1x02_P2.54mm_Vertical, symbol Connector:Conn_01x02_Female
- SW4: footprint Connector_Molex:Molex_SL_171971-0002_1x02_P2.54mm_Vertical -> TerminalBlock:TerminalBlock_bornier-2_P5.08mm
Connections:
- net labels removed: 12V_GND, BATT_GND, CAN_H, CAN_L, Memory
- wire segments 103 -> 80
- no-connect marks 2 -> 0
Other:
- note added: "From: https://kellycontroller.com/wp-content/uploads/kls-h/KLS-DHMN-CAD-Model-1130.pdf"
- note added: "Look to initial commit to see wiring and headers for connection \nstraight to controller connectors\n"
- note added: "Power to conactor coil"
- note added: "Rev 2: \nTo be used with Kelly assemblies on first prototype vehicle for basic manual control. \nFuture versions will use mcu\n\nChanges:\n- Dropping display output \n- Matching wiring needs of assemblies (flat connector used by assembly)\nTo do:\n- Make consistent with assembly configuration\n- - Incorporate 2A fuse between switch and 48V (PWR)?\n- - Put fuses, contactor, ext. switch on schemati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"
- note removed: "2A fuse needs to go here"
- note removed: "48V comes in from 10A fuse on assembly\n"
- note removed: "48V from battery \npowers controller"
- note removed: "Images are looking into \nconnectors from board"
- note removed: "Kelly1:\n- Pin 12 – FWD (white)\n- Pin 6 - GND (black)\n- Pin 14 – REV SW (orange)\n- Pin 25 – Brake (yellow)\n- Pin 11 - 12V (red)\n- Pin 33 – CAN_H (green)\n- Pin 34 – CAN_L (brown)\n- Pin 7 – PWR (pink; purple from board)\nKelly2:\n- Pin 4 – 5V (purple)\n- Pin 2 – Brake_AN (brown)\n- Pin 20 – GND (black)\n- Pin 3 – Throttle (green)\n- Pin 15 – Foot_SW (gray)\n- Pin 8 – Meter (gray; white on bo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"
- note removed: "Rev 2: \nTo be used with Kelly assemblies on first prototype vehicle for basic manual control. \nFuture versions will use mcu\n\nChanges:\n- Dropping display output \n- Matching wiring needs of assemblies\nTo do:\n- Remove display components\n- - Header\n- - 48V line ('memory') from battery? (Keep as header?)\n- Make consistent with assembly configuration\n- - Incorporate 2A fuse between switch a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"

Commit message: PCB routed and ready for cutting
Other:
- note added: "J2 connections:\n1: +48V\n2: +12V\n3: Foot_SW\n4: Brake (12V)\n5: REV\n6: FWD\n7: 5V\n8: Throttle\n9: Brake_AN\n10: Meter\n11: PWR\n12: GND"
Changed lines of the file:
@@
 $EndComp
-Wire Wire Line
-	6750 2000 6750 2850
 Wire Wire Line
 	6750 2850 7300 2850
@@
 Connection ~ 6650 2950
 Wire Wire Line
-	6750 2850 6750 3000
-Wire Wire Line
-	6750 3000 6250 3000
-Connection ~ 6750 2850
-Wire Wire Line
 	6850 2750 6850 3100
 Wire Wire Line
@@
 	6450 2150 6450 2200
 Wire Wire Line
-	6450 2200 6250 2200
-Wire Wire Line
 	6450 2150 7300 2150
 Wire Wire Line
-	6250 2300 6450 2300
-Wire Wire Line
-	6450 2300 6450 2250
-Wire Wire Line
-	6450 2250 7300 2250
-Wire Wire Line
-	6250 2400 6450 2400
-Wire Wire Line
-	6450 2400 6450 2450
-Wire Wire Line
-	6450 2450 7300 2450
-Wire Wire Line
-	6250 2500 6450 2500
-Wire Wire Line
-	6450 2500 6450 2550
+	6350 2450 7300 2450
 Wire Wire Line
 	6450 2550 7300 2550
 Wire Wire Line
-	6250 2600 6450 2600
-Wire Wire Line
-	6450 2600 6450 2650
-Wire Wire Line
 	6450 2650 7300 2650
 Wire Wire Line
-	6450 3050 6450 2700
-Wire Wire Line
-	6450 2700 6250 2700
+	6450 3050 6450 3000
 Wire Wire Line
 	6450 3050 7300 3050
 Wire Wire Line
-	6500 3150 6500 2800
+	6550 3150 7300 3150
 Wire Wire Line
-	6500 2800 6250 2800
-Wire Wire Line
-	6500 3150 7300 3150
-Wire Wire Line
-	6400 3250 6400 2900
-Wire Wire Line
-	6400 2900 6250 2900
+	6400 3250 6400 2300
 Wire Wire Line
 	6400 3250 7300 3250
@@
 Wire Wire Line
 	4900 1500 4900 1700
+Wire Wire Line
+	6450 3000 6250 3000
+Wire Wire Line
+	6450 2900 6250 2900
+Wire Wire Line
+	6450 2900 6450 2650
+Wire Wire Line
+	6350 2800 6350 2450
+Wire Wire Line
+	6350 2800 6250 2800
+Wire Wire Line
+	6250 2700 6500 2700
+Wire Wire Line
+	6500 2700 6500 2250
+Wire Wire Line
+	6500 2250 7300 2250
+Wire Wire Line
+	6750 2000 6750 2600
+Wire Wire Line
+	6250 2600 6750 2600
+Connection ~ 6750 2600
+Wire Wire Line
+	6750 2600 6750 2850
+Wire Wire Line
+	6250 2300 6400 2300
+Wire Wire Line
+	6250 2200 6450 2200
+Text Notes 6100 4400 0    50   ~ 0
+J2 connections:\n1: +48V\n2: +12V\n3: Foot_SW\n4: Brake (12V)\n5: REV\n6: FWD\n7: 5V\n8: Throttle\n9: Brake_AN\n10: Meter\n11: PWR\n12: GND
+Wire Wire Line
+	6550 2400 6550 3150
+Wire Wire Line
+	6450 2500 6450 2550
+Wire Wire Line
+	6250 2500 6450 2500
+Wire Wire Line
+	6250 2400 6550 2400
 $EndSCHEMATC

Commit message: Split 12 pin connector realized did not have 12 pin connector so split roughly into power and controls cables redid pcb layout and exported gerbers;
Parts:
- removed J2: Conn_01x12_Female, Connector_Molex:Molex_SL_171971-0012_1x12_P2.54mm_Vertical, symbol Connector:Conn_01x12_Female
- added J1, J2: Conn_01x06_Female, Connector_Molex:Molex_SL_171971-0006_1x06_P2.54mm_Vertical, symbol Connector:Conn_01x06_Female
- H1, H2, H3, H4: footprint MountingHole:MountingHole_3.2mm_M3_ISO14580 -> myfootprints:MountingHole_3.2mm_M3_through_hole
Connections:
- wire segments 80 -> 81
Other:
- note added: "KC connections:\nJ1:\n 1: Foot_SW\n 2: Brake (12V)\n 3: REV\n 4: FWD\n 5: Brake_AN\n 6: Throttle\nJ2:\n 1: PWR\n 2: +48V\n 3: +12V\n 4: + 5V\n 5: GND\n 6: Meter"
- note added: "Rev 2: \nTo be used with Kelly assemblies on first prototype vehicle for basic manual control. \nFuture versions will use mcu\n\nChanges:\n- Dropping display output \n- Matching wiring needs of assemblies (flat connector used by assembly)\nTo do:\n\nURLs:\n- KLS controller manual: https://kellycontroller.com/wp-content/uploads/kls-nm/KellyKLS-N-UserManualV2.7.pdf\n- Control box and assembly schem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"
- note removed: "J2 connections:\n1: +48V\n2: +12V\n3: Foot_SW\n4: Brake (12V)\n5: REV\n6: FWD\n7: 5V\n8: Throttle\n9: Brake_AN\n10: Meter\n11: PWR\n12: GND"
- note removed: "Rev 2: \nTo be used with Kelly assemblies on first prototype vehicle for basic manual control. \nFuture versions will use mcu\n\nChanges:\n- Dropping display output \n- Matching wiring needs of assemblies (flat connector used by assembly)\nTo do:\n- Make consistent with assembly configuration\n- - Incorporate 2A fuse between switch and 48V (PWR)?\n- - Put fuses, contactor, ext. switch on schemati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"
Changed lines of the file:
@@
 F 0 "H1" H 850 2746 50  0000 L CNN
 F 1 "MountingHole" H 850 2655 50  0000 L CNN
-F 2 "MountingHole:MountingHole_3.2mm_M3_ISO14580" H 750 2700 50  0001 C CNN
+F 2 "myfootprints:MountingHole_3.2mm_M3_through_hole" H 750 2700 50  0001 C CNN
 F 3 "~" H 750 2700 50  0001 C CNN
 	1    750  2700
@@
 F 0 "H2" H 850 3096 50  0000 L CNN
 F 1 "MountingHole" H 850 3005 50  0000 L CNN
-F 2 "MountingHole:MountingHole_3.2mm_M3_ISO14580" H 750 3050 50  0001 C CNN
+F 2 "myfootprints:MountingHole_3.2mm_M3_through_hole" H 750 3050 50  0001 C CNN
 F 3 "~" H 750 3050 50  0001 C CNN
 	1    750  3050
@@
 F 0 "H3" H 850 3446 50  0000 L CNN
 F 1 "MountingHole" H 850 3355 50  0000 L CNN
-F 2 "MountingHole:MountingHole_3.2mm_M3_ISO14580" H 750 3400 50  0001 C CNN
+F 2 "myfootprints:MountingHole_3.2mm_M3_through_hole" H 750 3400 50  0001 C CNN
 F 3 "~" H 750 3400 50  0001 C CNN
 	1    750  3400
@@
 F 0 "H4" H 850 3796 50  0000 L CNN
 F 1 "MountingHole" H 850 3705 50  0000 L CNN
-F 2 "MountingHole:MountingHole_3.2mm_M3_ISO14580" H 750 3750 50  0001 C CNN
+F 2 "myfootprints:MountingHole_3.2mm_M3_through_hole" H 750 3750 50  0001 C CNN
 F 3 "~" H 750 3750 50  0001 C CNN
 	1    750  3750
@@
 make sure boost is not\nenabled in app
 Text Notes 650  7750 0    100  ~ 0
-Rev 2: \nTo be used with Kelly assemblies on first prototype vehicle for basic manual control. \nFuture versions will use mcu\n\nChanges:\n- Dropping display output \n- Matching wiring needs of assemblies (flat connector used by assembly)\nTo do:\n- Make consistent with assembly configuration\n- -  Incorporate 2A fuse between switch and 48V (PWR)?\n- - Put fuses, contactor, ext. switch on schematic\n- - - Use number sign in front of reference so they don't show up on PCB\n- Use bigger board connector for switch\n\nURLs:\n- KLS controller manual: https://kellycontroller.com/wp-content/uploads/kls-nm/KellyKLS-N-UserManualV2.7.pdf\n- Control box and assembly schematic: https://kellycontroller.com/wp-content/uploads/kls-h/KLS-DHMN-CAD-Model-1130.pdf\n- Display datasheet: https://drive.google.com/file/d/12TWD7V3HLI8IPtFdbf37xQo0YPuW2e0G/view
+Rev 2: \nTo be used with Kelly assemblies on first prototype vehicle for basic manual control. \nFuture versions will use mcu\n\nChanges:\n- Dropping display output \n- Matching wiring needs of assemblies (flat connector used by assembly)\nTo do:\n\nURLs:\n- KLS controller manual: https://kellycontroller.com/wp-content/uploads/kls-nm/KellyKLS-N-UserManualV2.7.pdf\n- Control box and assembly schematic: https://kellycontroller.com/wp-content/uploads/kls-h/KLS-DHMN-CAD-Model-1130.pdf\n- Display datasheet: https://drive.google.com/file/d/12TWD7V3HLI8IPtFdbf37xQo0YPuW2e0G/view
 Text Notes 7000 1750 0    50   ~ 0
 From: https://kellycontroller.com/wp-content/uploads/kls-h/KLS-DHMN-CAD-Model-1130.pdf
@@
 $EndComp
 Wire Wire Line
-	6950 3400 6950 2350
-Wire Wire Line
 	6950 2350 7300 2350
 Text Label 7150 2250 0    50   ~ 0
 FWD
-$Comp
-L Connector:Conn_01x12_Female J2
-U 1 1 6196588F
-P 6050 2700
-F 0 "J2" H 5942 1875 50  0000 C CNN
-F 1 "Conn_01x12_Female" H 5942 1966 50  0000 C CNN
-F 2 "Connector_Molex:Molex_SL_171971-0012_1x12_P2.54mm_Vertical" H 6050 2700 50  0001 C CNN
-F 3 "~" H 6050 2700 50  0001 C CNN
-	1    6050 2700
-	-1   0    0    1
-$EndComp
-Wire Wire Line
-	6650 2950 6650 3200
-Wire Wire Line
-	6650 3200 6250 3200
 Connection ~ 6650 2950
-Wire Wire Line
-	6850 2750 6850 3100
-Wire Wire Line
-	6850 3100 6250 3100
 Connection ~ 6850 2750
-Wire Wire Line
-	6950 2350 6550 2350
-Wire Wire Line
-	6550 2350 6550 2100
-Wire Wire Line
-	6550 2100 6250 2100
-Connection ~ 6950 2350
-Wire Wire Line
-	6450 2150 6450 2200
-Wire Wire Line
-	6450 2150 7300 2150
-Wire Wire Line
-	6350 2450 7300 2450
-Wire Wire Line
-	6450 2550 7300 2550
-Wire Wire Line
-	6450 2650 7300 2650
-Wire Wire Line
-	6450 3050 6450 3000
-Wire Wire Line
-	6450 3050 7300 3050
-Wire Wire Line
-	6550 3150 7300 3150
-Wire Wire Line
-	6400 3250 6400 2300
-Wire Wire Line
-	6400 3250 7300 3250
 Connection ~ 7800 800
 Wire Wire Line
@@
 Wire Wire Line
 	4900 1500 4900 1700
+Text Notes 6050 4800 0    50   ~ 0
+KC connections:\nJ1:\n 1: Foot_SW\n 2: Brake (12V)\n 3: REV\n 4: FWD\n 5: Brake_AN\n 6: Throttle\nJ2:\n 1: PWR\n 2: +48V\n 3: +12V\n 4: + 5V\n 5: GND\n 6: Meter
+Wire Wire Line
+	6750 2000 6750 2850
+$Comp
+L Connector:Conn_01x06_Female J1
+U 1 1 61A47E49
+P 6000 2300
+F 0 "J1" H 5892 1775 50  0000 C CNN
+F 1 "Conn_01x06_Female" H 5892 1866 50  0000 C CNN
+F 2 "Connector_Molex:Molex_SL_171971-0006_1x06_P2.54mm_Vertical" H 6000 2300 50  0001 C CNN
+F 3 "~" H 6000 2300 50  0001 C CNN
+	1    6000 2300
+	-1   0    0    1
+$EndComp
+Wire Wire Line
+	6650 2950 6650 3300
+Wire Wire Line
+	6550 3150 7300 3150
+Wire Wire Line
+	6750 3100 6750 2850
+Connection ~ 6750 2850
+Wire Wire Line
+	7100 2150 7300 2150
+Wire Wire Line
+	6200 2500 6450 2500
+Wire Wire Line
+	6450 2500 6450 3050
+Wire Wire Line
+	6450 3050 7150 3050
+Wire Wire Line
+	7000 2400 7000 2650
+Wire Wire Line
+	7000 2650 7300 2650
+Wire Wire Line
+	6200 2300 6800 2300
+Wire Wire Line
+	6800 2300 6800 2450
+Wire Wire Line
+	6800 2450 7300 2450
+Wire Wire Line
+	6200 2200 7000 2200
+Wire Wire Line
+	7000 2200 7000 2250
+Wire Wire Line
+	7000 2250 7300 2250
+Wire Wire Line
+	6700 2550 7300 2550
+Wire Wire Line
+	6200 2400 7000 2400
+Wire Wire Line
+	6550 2100 6550 3150
+$Comp
+L Connector:Conn_01x06_Female J2
+U 1 1 61A8ECFC
+P 6000 3200
+F 0 "J2" H 5892 2675 50  0000 C CNN
+F 1 "Conn_01x06_Female" H 5892 2766 50  0000 C CNN
+F 2 "Connector_Molex:Molex_SL_171971-0006_1x06_P2.54mm_Vertical" H 6000 3200 50  0001 C CNN
+F 3 "~" H 6000 3200 50  0001 C CNN
+	1    6000 3200
+	-1   0    0    1
+$EndComp
 Wire Wire Line
-	6450 3000 6250 3000
+	7050 3250 7400 3250
 Wire Wire Line
-	6450 2900 6250 2900
+	7100 2150 7100 3350
 Wire Wire Line
-	6450 2900 6450 2650
+	6850 2750 6850 3200
 Wire Wire Line
-	6350 2800 6350 2450
+	6200 3200 6850 3200
 Wire Wire Line
-	6350 2800 6250 2800
+	6200 3100 6750 3100
 Wire Wire Line
-	6250 2700 6500 2700
+	6200 3300 6650 3300
 Wire Wire Line
-	6500 2700 6500 2250
+	6200 3400 6750 3400
 Wire Wire Line
-	6500 2250 7300 2250
+	6750 3400 6750 3350
 Wire Wire Line
-	6750 2000 6750 2600
+	6750 3350 7100 3350
 Wire Wire Line
-	6250 2600 6750 2600
-Connection ~ 6750 2600
+	6950 2350 6950 3000
 Wire Wire Line
-	6750 2600 6750 2850
+	6200 2900 7050 2900
 Wire Wire Line
-	6250 2300 6400 2300
+	7050 2900 7050 3250
 Wire Wire Line
-	6250 2200 6450 2200
-Text Notes 6100 4400 0    50   ~ 0
-J2 connections:\n1: +48V\n2: +12V\n3: Foot_SW\n4: Brake (12V)\n5: REV\n6: FWD\n7: 5V\n8: Throttle\n9: Brake_AN\n10: Meter\n11: PWR\n12: GND
+	6200 3000 6950 3000
+Connection ~ 6950 3000
 Wire Wire Line
-	6550 2400 6550 3150
+	6950 3000 6950 3400
 Wire Wire Line
-	6450 2500 6450 2550
+	6200 2100 6550 2100
 Wire Wire Line
-	6250 2500 6450 2500
+	6200 2000 6700 2000
 Wire Wire Line
-	6250 2400 6550 2400
+	6700 2000 6700 2550
 $EndSCHEMATC

Commit message: first board cut and connected successfully
some minor changes to make before cutting second board, including removing battery connector and flipping some connectors
Other:
- note added: "KC connections:\nJ1:\n 1: Foot_SW (blue)\n 2: Brake (12v / gray)\n 3: REV (purple)\n 4: FWD (yellow)\n 5: Brake_AN (green)\n 6: Throttle (white)\nJ2:\n 1: PWR (brown)\n 2: +48V (orange)\n 3: +12V (thick red)\n 4: + 5V (red)\n 5: GND (black)\n 6: Meter (dark gray)\n"
- note added: "Rev 2: \nTo be used with Kelly assemblies on first prototype vehicle for basic manual control. \nFuture versions will use mcu\n\nChanges:\n- Dropped display output \n- Adapted wiring to flat 14 pin connector from assembly\nTo do:\n- Remove Batt connector (superfluous - power comes in on brown line and goes back to \n controller on pink line via power switch)\n- Flip control connectors to face sam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"
- note removed: "KC connections:\nJ1:\n 1: Foot_SW\n 2: Brake (12V)\n 3: REV\n 4: FWD\n 5: Brake_AN\n 6: Throttle\nJ2:\n 1: PWR\n 2: +48V\n 3: +12V\n 4: + 5V\n 5: GND\n 6: Meter"
- note removed: "Rev 2: \nTo be used with Kelly assemblies on first prototype vehicle for basic manual control. \nFuture versions will use mcu\n\nChanges:\n- Dropping display output \n- Matching wiring needs of assemblies (flat connector used by assembly)\nTo do:\n\nURLs:\n- KLS controller manual: https://kellycontroller.com/wp-content/uploads/kls-nm/KellyKLS-N-UserManualV2.7.pdf\n- Control box and assembly schem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"

Commit message: Ready to cut second board
Thickened 12V traces and removed batt connector which was superfluous
Parts:
- removed J3: Batt, TerminalBlock:TerminalBlock_bornier-2_P5.08mm, symbol Connector:Conn_01x02_Female
Connections:
- wire segments 81 -> 79
Other:
- note added: "Brn Yell RED Whi Grn Prpl \n\n\n\n\n\n\nOrng Drk Red Blk Blu\n gry"
- note added: "Rev 2: \nTo be used with Kelly assemblies on first prototype vehicle for basic manual control. \nFuture versions will use mcu\n\nChanges:\n- Dropped display output \n- Adapted wiring to flat 14 pin connector from assembly\n- Dropped battery connector (superfluous - power comes in on brown line and goes back to \n controller on pink line via power switch)\n- Made 12V line thicker (consistent with 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"
- note removed: "Power to conactor coil"
- note removed: "Rev 2: \nTo be used with Kelly assemblies on first prototype vehicle for basic manual control. \nFuture versions will use mcu\n\nChanges:\n- Dropped display output \n- Adapted wiring to flat 14 pin connector from assembly\nTo do:\n- Remove Batt connector (superfluous - power comes in on brown line and goes back to \n controller on pink line via power switch)\n- Flip control connectors to face sam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"

Commit message: saving most recent changes in preparation for moving to mcu based schematics
Other:
- note added: "Pins needed for MCU board:\nSPI: 4 (if using quad digital pot. Otherwise more)\nI2C: 2\n(Pot inputs:2 - unless using i2c rotation sensor)\nBrake button inputs: 2\nBrake signal outputs: 2\nMeter input: 1"
Changed lines of the file:
@@
 Text Notes 7900 5450 0    50   ~ 0
 Brn   Yell RED  Whi Grn  Prpl \n\n\n\n\n\n\nOrng Drk Red  Blk  Blu\n     gry
+Text Notes 200  1150 0    50   ~ 0
+Pins needed for MCU board:\nSPI: 4 (if using quad digital pot. Otherwise more)\nI2C: 2\n(Pot inputs:2 - unless using i2c rotation sensor)\nBrake button inputs: 2\nBrake signal outputs: 2\nMeter input: 1
 $EndSCHEMATC

Commit message: redid board. vias were too small and close together. Also changed many pads to oval
Parts:
- removed J4: Meter, Connector_Molex:Molex_SL_171971-0002_1x02_P2.54mm_Vertical, symbol Connector:Conn_01x02_Female
- removed RV2: Brake, Connector_Molex:Molex_SL_171971-0003_1x03_P2.54mm_Vertical, symbol Device:R_POT
- removed SW2: Foot Switch, Connector_Molex:Molex_SL_171971-0002_1x02_P2.54mm_Vertical, symbol Switch:SW_SPST
- removed SW3: Brake, Connector_Molex:Molex_SL_171971-0002_1x02_P2.54mm_Vertical, symbol Switch:SW_SPST
- added B1: SPARKFUN_PRO_MICRO, Boards:SPARKFUN_PRO_MICRO, symbol SparkFun-Boards:SPARKFUN_PRO_MICRO
- added J10: 48V, Connector_Molex:Molex_SL_171971-0002_1x02_P2.54mm_Vertical, symbol Connector:Conn_01x02_Female
- added J11, J12: Conn_01x06_Female, Connector_Molex:Molex_SL_171971-0006_1x06_P2.54mm_Vertical, symbol Connector:Conn_01x06_Female
- added J3: I2C throttle, Connector_Molex:Molex_SL_171971-0004_1x04_P2.54mm_Vertical, symbol Connector:Conn_01x04_Female
- added J8: 12V, Connector_Molex:Molex_SL_171971-0002_1x02_P2.54mm_Vertical, symbol Connector:Conn_01x02_Female
- added J9: 5V, Connector_Molex:Molex_SL_171971-0002_1x02_P2.54mm_Vertical, symbol Connector:Conn_01x02_Female
- added R1, R2, R8: 1k, Resistor_THT:R_Axial_DIN0207_L6.3mm_D2.5mm_P7.62mm_Horizontal, symbol Device:R
- added R3, R4, R5: 220, Resistor_THT:R_Axial_DIN0207_L6.3mm_D2.5mm_P7.62mm_Horizontal, symbol Device:R
- added R6, R7: 10k, Resistor_THT:R_Axial_DIN0207_L6.3mm_D2.5mm_P7.62mm_Horizontal, symbol Device:R
- added SW2: SW_Push, Connector_Molex:Molex_SL_171971-0002_1x02_P2.54mm_Vertical, symbol Switch:SW_Push
- added SW5: Power Switch, TerminalBlock:TerminalBlock_bornier-2_P5.08mm, symbol Switch:SW_SPST
- added U1, U2: LTV-247, Package_DIP:DIP-16_W7.62mm_LongPads, symbol Isolator:LTV-247
- added U3: MCP4251-xxxx-P, Package_DIP:DIP-14_W7.62mm, symbol Potentiometer_Digital:MCP4251-xxxx-P
Connections:
- net labels added: +12VA, +48VA, +5VA, 10-CS, 12V-A, 5-Forward, 5V-A, 6-Reverse, 8-Meter, 9-Meter, Brake-A, Brake_AN-A, FWD-A, Foot_SW-A, GNDA, Meter-A, PWR-A, REV-A, Throttle-A, VCC
- wire segments 79 -> 234
- no-connect marks 0 -> 13
Other:
- note added: "Arduino Pro Micro connections:\n- SPI: 15 (SCK), 16 (MOSI), 14 (MISO), 10 (CS - "motorsPin")\n- I2C: 2 (SDA), 3 (SCL)\n- Meter pins: 8, 9\n- brakes pin: 7\n- Reverse pin: 6\n- Forward pin: 5\n- Throttle pot pin: A0"
- note added: "Contactor is energized along with \nKelly controller when power\nswitch is engaged\nMounted off board"
- note added: "KC connections:\nJ1/J11:\n 1: Foot_SW (blue)\n 2: Brake (12v / gray)\n 3: REV (purple)\n 4: FWD (yellow)\n 5: Brake_AN (green)\n 6: Throttle (white)\nJ2/J12:\n 1: PWR (brown)\n 2: +48V (orange)\n 3: +12V (thick red)\n 4: + 5V (red)\n 5: GND (black)\n 6: Meter (dark gray)\n"
- note added: "MCU based dual Kelly controller interface board\n- Using Arduino pro micro\n- Concept is to keep Arduino and Kelly controllers electrically isolated\n except for MCU power\n - Electrical isolation accomplished by use of digital pot (mcp4251) for throttle \n and optocouplers for switches\n\nGeneral Notes:\n- meter signals are 12V\n\nBuild Notes:\n- Using mcp4251 not ltv247 opto as depicted\n- Not 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"
- note added: "To do:\nMock up 12V FR switches on opto"
- note removed: "Contactor is energizd along with \nKelly controller when power\nswitch is engaged"
- note removed: "KC connections:\nJ1:\n 1: Foot_SW (blue)\n 2: Brake (12v / gray)\n 3: REV (purple)\n 4: FWD (yellow)\n 5: Brake_AN (green)\n 6: Throttle (white)\nJ2:\n 1: PWR (brown)\n 2: +48V (orange)\n 3: +12V (thick red)\n 4: + 5V (red)\n 5: GND (black)\n 6: Meter (dark gray)\n"
- note removed: "Pins needed for MCU board:\nSPI: 4 (if using quad digital pot. Otherwise more)\nI2C: 2\n(Pot inputs:2 - unless using i2c rotation sensor)\nBrake button inputs: 2\nBrake signal outputs: 2\nMeter input: 1"
- note removed: "Rev 2: \nTo be used with Kelly assemblies on first prototype vehicle for basic manual control. \nFuture versions will use mcu\n\nChanges:\n- Dropped display output \n- Adapted wiring to flat 14 pin connector from assembly\n- Dropped battery connector (superfluous - power comes in on brown line and goes back to \n controller on pink line via power switch)\n- Made 12V line thicker (consistent with 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"
- note removed: "make sure boost is not\nenabled in app"
