File: Kelly controller.sch (KiCad schematic (older format))
At the start: 32 parts, among them J1 Conn_01x06_Female, J10 48V, J11 Conn_01x06_Female, J12 Conn_01x06_Female, J2 Conn_01x06_Female, J3 I2C throttle, J5 48V, J6 12V, J7 5V, J8 12V, J9 5V, SW1 FNR, SW2 Brake_SW, SW4 Power Switch, SW5 Power Switch, U1 LTV-247, U2 LTV-247, U3 MCP4251-xxxx-P

Commit message: Last version of mcp4251 based board. Too many problems but ultimately got to work by combining grounds and putting diodes in line with pot high side to get lower that Arduino Vcc. Next version will use PWM buffered by opamp
Parts:
- removed J10, J5: 48V, Connector_Molex:Molex_SL_171971-0002_1x02_P2.54mm_Vertical, symbol Connector:Conn_01x02_Female
- removed J7, J9: 5V, Connector_Molex:Molex_SL_171971-0002_1x02_P2.54mm_Vertical, symbol Connector:Conn_01x02_Female
- removed J8: 12V, Connector_Molex:Molex_SL_171971-0002_1x02_P2.54mm_Vertical, symbol Connector:Conn_01x02_Female
- added D1, D2: yellow, myfootprints:LED_D3.0mm_wide_pads, symbol Device:LED
- added D3, D4: green, myfootprints:LED_D3.0mm_wide_pads, symbol Device:LED
- added D5, D6: RED, myfootprints:LED_D3.0mm_wide_pads, symbol Device:LED
- added J4: throttle A, myfootprints:PinHeader_1x03_P2.54mm_Vertical_wide_pads, symbol Connector:Conn_01x03_Female
- added J5: throttle B, myfootprints:PinHeader_1x03_P2.54mm_Vertical_wide_pads, symbol Connector:Conn_01x03_Female
- added J7: B_5_12_48, myfootprints:PinHeader_1x04_P2.54mm_Vertical_wide_pads, symbol Connector:Conn_01x04_Female
- added J8: A_5_12_48, myfootprints:PinHeader_1x04_P2.54mm_Vertical_wide_pads, symbol Connector:Conn_01x04_Female
- added JP1: Jumper, Connector_PinHeader_2.54mm:PinHeader_1x02_P2.54mm_Vertical, symbol Device:Jumper
- added R10, R11, R12, R9: 1k, myfootprints:R_Axial_DIN0207_L6.3mm_D2.5mm_P7.62mm_Horizontal_wide_pads, symbol Device:R
- added TP1: RC, Connector_PinHeader_2.54mm:PinHeader_1x01_P2.54mm_Vertical, symbol Connector:TestPoint
- added TP12, TP13: ftsw, Connector_PinHeader_2.54mm:PinHeader_1x01_P2.54mm_Vertical, symbol Connector:TestPoint
- added TP14, TP15: anbrk, Connector_PinHeader_2.54mm:PinHeader_1x01_P2.54mm_Vertical, symbol Connector:TestPoint
- added U4: SPAN02C-05, myfootprints:SPAN02, symbol my_devices:SPAN02C-05
- J3: footprint Connector_Molex:Molex_SL_171971-0004_1x04_P2.54mm_Vertical -> myfootprints:Molex_SL_171971-0004_1x04_P2.54mm_Vertical_wide_pads
- J6: value 12V -> Board power; footprint Connector_Molex:Molex_SL_171971-0002_1x02_P2.54mm_Vertical -> Connector_PinHeader_2.54mm:PinHeader_1x02_P2.54mm_Vertical
- R1, R2, R3, R4, R5, R6, R7, R8: footprint Resistor_THT:R_Axial_DIN0207_L6.3mm_D2.5mm_P7.62mm_Horizontal -> myfootprints:R_Axial_DIN0207_L6.3mm_D2.5mm_P7.62mm_Horizontal_wide_pads
- RV1, SW1: footprint Connector_Molex:Molex_SL_171971-0003_1x03_P2.54mm_Vertical -> myfootprints:Molex_SL_171971-0003_1x03_P2.54mm_Vertical_wide_pads
- U3: value MCP4251-xxxx-P -> MCP4251
Connections:
- net labels added: +12VB, +48VB, +5VB, 5-Reverse, 6-Forward, 8-Meter_A, 9-Meter_B, Brake-B, Brake_AN-B, FWD-B, Foot_SW-B, GNDB, Meter-B, PWR-B, REV-B, Throttle-B
- net labels removed: +48V, 12V, 12V-A, 5-Forward, 5V-A, 6-Reverse, 8-Meter, 9-Meter, Brake, Brake_AN, FWD, Foot_SW, Meter, PWR, REV, Throttle
- wire segments 234 -> 280
- no-connect marks 13 -> 8
Other:
- note added: "Arduino Pro Micro connections:\n- SPI: 15 (SCK), 16 (MOSI), 14 (MISO), 10 (CS - "motorsPin")\n- I2C: 2 (SDA), 3 (SCL)\n- Meter pins: 8 (A), 9 (B)\n- brakes pin: 7\n- Forward pin: 6\n- Reverse pin: 5\n- Throttle pot pin: A0"
- note added: "Contactor is energized along with \nKelly controller when power\nswitch is engaged.\nMounted off board"
- note added: "Kelly controller connections:\n5VA and 5VB connect - pin 4 (5V)\nGNDA and GNDB connect - pin 6 (GND)\nThrottle lines - pin 3 (Throttle)"
- note added: "Troubleshooting notes:\n5/1/22: Wired up new board. Brake and FNR work fine. Throttle is not working properly. Motors run even when\npot turned all the way down. Pot output behaves as it should when connected alone to laptop. Output\nvalues were all over the place when working in the garage. Problem persisted even when motors were \ndisconnected. Need to try again in garage with laptop connected.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"
- note removed: "Arduino Pro Micro connections:\n- SPI: 15 (SCK), 16 (MOSI), 14 (MISO), 10 (CS - "motorsPin")\n- I2C: 2 (SDA), 3 (SCL)\n- Meter pins: 8, 9\n- brakes pin: 7\n- Reverse pin: 6\n- Forward pin: 5\n- Throttle pot pin: A0"
- note removed: "Contactor is energized along with \nKelly controller when power\nswitch is engaged\nMounted off board"
- note removed: "Fix this after saving in git\n--> should be 12v over Brake"
- note removed: "Need to add Vcc line\nin next version"
- note removed: "Troubleshooting notes:\n4/16/22: First single board dual controller prototype\n- Tested with Arduino power side only. After updating pin assignments throttle worked. No response from brake or FNR. Connected both \nmotors. Both systems powered up, but motors didn't run in sync. Found that voltage into digital pot on J1/J2 side was lower than J11/J12 side, resulting in different Vout from digital p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"
- note removed: "Vcc line got orphaned\n- Need to fix"

Commit message: Getting ready to move on to new version without digital pots. Added some notes re. how got last board to work. Added jumpers to tie grounds together. Next version will be dead simple dual pot board. If implementing mcu will probably use pwm to opamp buffer.
Parts:
- added JP? (x2): Jumper, Connector_PinHeader_2.54mm:PinHeader_1x02_P2.54mm_Vertical, symbol Device:Jumper
Connections:
- wire segments 280 -> 288
Other:
- note added: "Haven't decided yet on best way to tie grounds together\n"
- note added: "Switched 5VA and 5VB to Vcc on pot connections.\nHaven't tested. To get last cut board to work \ncut traces and put diodes in line. Voltage drop\nseems to have done the trick."
Changed lines of the file:
@@
 Throttle-A
 $Comp
-L power:+5VA #PWR025
-U 1 1 627F88BE
-P 7550 5300
-F 0 "#PWR025" H 7550 5150 50  0001 C CNN
-F 1 "+5VA" H 7650 5350 50  0000 C CNN
-F 2 "" H 7550 5300 50  0001 C CNN
-F 3 "" H 7550 5300 50  0001 C CNN
-	1    7550 5300
-	1    0    0    -1
-$EndComp
-$Comp
 L Device:R R1
 U 1 1 624A6209
@@
 $EndComp
 $Comp
-L my_devices:+5VB #PWR030
-U 1 1 62FE6574
-P 7550 4900
-F 0 "#PWR030" H 7550 4750 50  0001 C CNN
-F 1 "+5VB" H 7650 5000 50  0000 C CNN
-F 2 "" H 7550 4900 50  0001 C CNN
-F 3 "" H 7550 4900 50  0001 C CNN
-	1    7550 4900
-	1    0    0    -1
-$EndComp
-$Comp
 L my_devices:GNDB #PWR029
 U 1 1 62FE877D
@@
 Text Notes 8050 4650 0    50   ~ 0
 Kelly controller connections:\n5VA and 5VB connect - pin 4 (5V)\nGNDA and GNDB connect - pin 6 (GND)\nThrottle lines - pin 3 (Throttle)
+$Comp
+L Device:Jumper JP?
+U 1 1 628C9383
+P 8400 2500
+F 0 "JP?" H 8400 2764 50  0000 C CNN
+F 1 "Jumper" H 8400 2673 50  0000 C CNN
+F 2 "Connector_PinHeader_2.54mm:PinHeader_1x02_P2.54mm_Vertical" H 8400 2500 50  0001 C CNN
+F 3 "~" H 8400 2500 50  0001 C CNN
+	1    8400 2500
+	1    0    0    -1
+$EndComp
+$Comp
+L Device:Jumper JP?
+U 1 1 628CF9D3
+P 8400 2900
+F 0 "JP?" H 8400 3164 50  0000 C CNN
+F 1 "Jumper" H 8400 3073 50  0000 C CNN
+F 2 "Connector_PinHeader_2.54mm:PinHeader_1x02_P2.54mm_Vertical" H 8400 2900 50  0001 C CNN
+F 3 "~" H 8400 2900 50  0001 C CNN
+	1    8400 2900
+	1    0    0    -1
+$EndComp
+$Comp
+L power:GND #PWR?
+U 1 1 628D0193
+P 7900 3200
+F 0 "#PWR?" H 7900 2950 50  0001 C CNN
+F 1 "GND" H 7905 3027 50  0000 C CNN
+F 2 "" H 7900 3200 50  0001 C CNN
+F 3 "" H 7900 3200 50  0001 C CNN
+	1    7900 3200
+	1    0    0    -1
+$EndComp
+Wire Wire Line
+	8100 2500 7900 2500
+Wire Wire Line
+	7900 2500 7900 2900
+Wire Wire Line
+	8100 2900 7900 2900
+Connection ~ 7900 2900
+Wire Wire Line
+	7900 2900 7900 3200
+$Comp
+L power:GNDA #PWR?
+U 1 1 629030A9
+P 9100 2650
+F 0 "#PWR?" H 9100 2400 50  0001 C CNN
+F 1 "GNDA" H 9105 2477 50  0000 C CNN
+F 2 "" H 9100 2650 50  0001 C CNN
+F 3 "" H 9100 2650 50  0001 C CNN
+	1    9100 2650
+	1    0    0    -1
+$EndComp
+Wire Wire Line
+	8700 2500 9100 2500
+Wire Wire Line
+	9100 2500 9100 2650
+$Comp
+L my_devices:GNDB #PWR?
+U 1 1 6291EA55
+P 9100 3150
+F 0 "#PWR?" H 9100 2900 50  0001 C CNN
+F 1 "GNDB" H 9105 2977 50  0000 C CNN
+F 2 "" H 9100 3150 50  0001 C CNN
+F 3 "" H 9100 3150 50  0001 C CNN
+	1    9100 3150
+	1    0    0    -1
+$EndComp
+Wire Wire Line
+	8700 2900 9100 2900
+Wire Wire Line
+	9100 2900 9100 3150
+Text Notes 7750 3500 0    50   ~ 0
+Haven't decided yet on best way to tie grounds together\n
+$Comp
+L power:VCC #PWR?
+U 1 1 6295971A
+P 7550 4900
+F 0 "#PWR?" H 7550 4750 50  0001 C CNN
+F 1 "VCC" H 7565 5073 50  0000 C CNN
+F 2 "" H 7550 4900 50  0001 C CNN
+F 3 "" H 7550 4900 50  0001 C CNN
+	1    7550 4900
+	1    0    0    -1
+$EndComp
+$Comp
+L power:VCC #PWR?
+U 1 1 62959E41
+P 7550 5300
+F 0 "#PWR?" H 7550 5150 50  0001 C CNN
+F 1 "VCC" H 7565 5473 50  0000 C CNN
+F 2 "" H 7550 5300 50  0001 C CNN
+F 3 "" H 7550 5300 50  0001 C CNN
+	1    7550 5300
+	1    0    0    -1
+$EndComp
+Text Notes 7300 6000 0    50   ~ 0
+Switched 5VA and 5VB to Vcc on pot connections.\nHaven't tested. To get last cut board to work \ncut traces and put diodes in line. Voltage drop\nseems to have done the trick.
 $EndSCHEMATC

Commit message: Dropping Arduino and digital pot. Using dual pot for control. This way can have total isolation between Kelly controllers. Currently have optoisolators in place for brake and FNR control. May switch with relays before cutting board. Expect to eventually return to MCU based board, but want something dead simple for prototyping.
Parts:
- removed B1: SPARKFUN_PRO_MICRO, Boards:SPARKFUN_PRO_MICRO, symbol SparkFun-Boards:SPARKFUN_PRO_MICRO
- removed J3: I2C throttle, myfootprints:Molex_SL_171971-0004_1x04_P2.54mm_Vertical_wide_pads, symbol Connector:Conn_01x04_Female
- removed J4: throttle A, myfootprints:PinHeader_1x03_P2.54mm_Vertical_wide_pads, symbol Connector:Conn_01x03_Female
- removed J5: throttle B, myfootprints:PinHeader_1x03_P2.54mm_Vertical_wide_pads, symbol Connector:Conn_01x03_Female
- removed R6, R7: 10k, myfootprints:R_Axial_DIN0207_L6.3mm_D2.5mm_P7.62mm_Horizontal_wide_pads, symbol Device:R
- removed U3: MCP4251, Package_DIP:DIP-14_W7.62mm, symbol Potentiometer_Digital:MCP4251-xxxx-P
- added D?: yellow, myfootprints:LED_D3.0mm_wide_pads, symbol Device:LED
- added JP?: pwr_jumper, symbol Jumper:Jumper_3_Bridged12
- added R?: 1k, myfootprints:R_Axial_DIN0207_L6.3mm_D2.5mm_P7.62mm_Horizontal_wide_pads, symbol Device:R
- added R?: 2.2k, myfootprints:R_Axial_DIN0207_L6.3mm_D2.5mm_P7.62mm_Horizontal_wide_pads, symbol Device:R
- added RV?: throttle(10k), symbol Device:R_POT_Dual
- added RV?: trim(1k), myfootprints:Molex_SL_171971-0003_1x03_P2.54mm_Vertical_wide_pads, symbol Device:R_POT
- added TP?: T_A, Connector_PinHeader_2.54mm:PinHeader_1x01_P2.54mm_Vertical, symbol Connector:TestPoint
- added TP?: T_B, Connector_PinHeader_2.54mm:PinHeader_1x01_P2.54mm_Vertical, symbol Connector:TestPoint
- R11, R12: value 1k -> 2.2k
- RV1: value Throttle -> trim(1k)
Connections:
- net labels removed: 10-CS, 5-Reverse, 6-Forward, 7-Brake, 8-Meter_A, 9-Meter_B, SCL, SDA
- wire segments 288 -> 229
- no-connect marks 8 -> 0
Other:
- note added: "In case need to tie grounds together\n"
- note added: "Try powering off 5VA first"
- note removed: "Arduino Pro Micro connections:\n- SPI: 15 (SCK), 16 (MOSI), 14 (MISO), 10 (CS - "motorsPin")\n- I2C: 2 (SDA), 3 (SCL)\n- Meter pins: 8 (A), 9 (B)\n- brakes pin: 7\n- Forward pin: 6\n- Reverse pin: 5\n- Throttle pot pin: A0"
- note removed: "Haven't decided yet on best way to tie grounds together\n"
- note removed: "Kelly controller connections:\n5VA and 5VB connect - pin 4 (5V)\nGNDA and GNDB connect - pin 6 (GND)\nThrottle lines - pin 3 (Throttle)"
- note removed: "Switched 5VA and 5VB to Vcc on pot connections.\nHaven't tested. To get last cut board to work \ncut traces and put diodes in line. Voltage drop\nseems to have done the trick."

Commit message: board ready to cut
Parts:
- removed J6: Board power, Connector_PinHeader_2.54mm:PinHeader_1x02_P2.54mm_Vertical, symbol Connector:Conn_01x02_Female
- removed JP1, JP? (x2): Jumper, Connector_PinHeader_2.54mm:PinHeader_1x02_P2.54mm_Vertical, symbol Device:Jumper
- removed JP?: pwr_jumper, symbol Jumper:Jumper_3_Bridged12
- removed R4: 220, myfootprints:R_Axial_DIN0207_L6.3mm_D2.5mm_P7.62mm_Horizontal_wide_pads, symbol Device:R
- removed TP1: RC, Connector_PinHeader_2.54mm:PinHeader_1x01_P2.54mm_Vertical, symbol Connector:TestPoint
- removed U2: LTV-247, Package_DIP:DIP-16_W7.62mm_LongPads, symbol Isolator:LTV-247
- removed U4: SPAN02C-05, myfootprints:SPAN02, symbol my_devices:SPAN02C-05
- added H5, H6: STAND-OFF, Hardware:STAND-OFF, symbol SparkFun-Hardware:STAND-OFF
- added J1: FNR switch, Connector_Molex:Molex_SL_171971-0005_1x05_P2.54mm_Vertical, symbol Connector:Conn_01x05_Female
- added JP1: Jumper_2_Open, Connector_PinHeader_2.54mm:PinHeader_1x02_P2.54mm_Vertical, symbol Jumper:Jumper_2_Open
- added R1: 1k, myfootprints:R_Axial_DIN0207_L6.3mm_D2.5mm_P7.62mm_Horizontal_wide_pads, symbol Device:R
- R2: renamed from R3; value 220 -> 1k
- R3: renamed from R5; value 220 -> 1k
- RV1: footprint myfootprints:Molex_SL_171971-0003_1x03_P2.54mm_Vertical_wide_pads -> myfootprints:trimpot_breadboard_spacing
- RV2: renamed from RV?; footprint (none) -> Connector_PinHeader_2.54mm:PinHeader_1x06_P2.54mm_Vertical
- RV3: renamed from RV?; footprint myfootprints:Molex_SL_171971-0003_1x03_P2.54mm_Vertical_wide_pads -> myfootprints:trimpot_breadboard_spacing
- gave numbers to parts that had none: 5
- renumbered D3 to D2, D4 to D3, D2 to D4, D1 to D5, D5 to D7, J8 to J3, J7 to J4, J11 to J5, J12 to J6, J1 to J7, J2 to J8, R1 to R10, R8 to R11, R10 to R13, R9 to R14, R11 to R7, R12 to R8, R2 to R9, SW2 to SW1, SW1 to SW2, SW5 to SW3, TP12 to TP4, TP13 to TP5, TP14 to TP6, TP15 to TP7
Connections:
- net labels removed: 5V, GND, VCC
- wire segments 229 -> 202
- no-connect marks 0 -> 6
Other:
- note added: "Barebones dual motor control board. Using dual pots to enable complete isolation between controllers\n\nBuild Notes:\n- Not implementing analog brake or foot switch\n\nChanges:\n- Removed arduino and digital pot and saved to new branch - two_motors_no_Arduino\n\nNext steps:\n\nTo do:\n- Add fuses for power lines\n- Update board with fixed SPAN02C footprint (will need more room)\n- Consider replac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"
- note added: "FNR connector Pinout\n1 - 12V; Pin 1 (Black)\n2 - 12V; Pin 4 (Brown)\n3 - D; Pin 2 (White)\n4 - R; Pin 3 (Purple)\n5 - GND; Pin 5 (Green)"
- note added: "For power wire\nstrain relief"
- note added: "Only install one or the other\nFNR selector"
- note removed: "In case need to tie grounds together\n"
- note removed: "MCU based dual Kelly controller interface board\n- Using Arduino pro micro\n- Concept is to keep Arduino and Kelly controllers electrically isolated\n except for MCU power\n - Electrical isolation accomplished by use of digital pot (mcp4251) for throttle \n and optocouplers for switches\n\nGeneral Notes:\n- meter signals are 12V so have to be buffered somehow\n\nBuild Notes:\n- Using P52501-4 not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"
- note removed: "Troubleshooting notes:\n5/1/22: Wired up new board. Brake and FNR work fine. Throttle is not working properly. Motors run even when\npot turned all the way down. Pot output behaves as it should when connected alone to laptop. Output\nvalues were all over the place when working in the garage. Problem persisted even when motors were \ndisconnected. Need to try again in garage with laptop connected.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"
- note removed: "Try powering off 5VA first"
